File: speaker-switcher-remote.kicad_pcb (KiCad board)
At the start: 2 copper layers, 49.8 x 60 mm, 17 parts, among them M1 arduino-nano, Q1 TIP31C, Q2 TIP31C

Commit message: Updated with arduino src code
Parts:
- added REF**: MountingHole_3.2mm_M3, MountingHole:MountingHole_3.2mm_M3, F.Cu at (90.2, 119.5)
- added REF**: MountingHole_3.2mm_M3, MountingHole:MountingHole_3.2mm_M3, F.Cu at (134.2, 119.5)
- added REF**: MountingHole_3.2mm_M3, MountingHole:MountingHole_3.2mm_M3, F.Cu at (134.2, 65.5)
- added REF**: MountingHole_3.2mm_M3, MountingHole:MountingHole_3.2mm_M3, F.Cu at (90.2, 65.5)
Routing:
- net GNDREF: track 97.3 -> 101.1 mm
