File: speaker-switcher-remote.sch (KiCad schematic (older format))
At the start: 27 parts, among them M1 arduino-nano, Q1 2N2222, Q2 TIP31C, U1 LM7805_TO220

Commit message: Updated w/PNP output stage
Parts:
- removed Q2: TIP31C, Package_TO_SOT_THT:TO-220-3_Vertical, symbol Device:Q_NPN_BCE
- added Q3: 2N2222, Package_TO_SOT_THT:TO-92, symbol Device:Q_NPN_EBC
- added Q4: Q_PNP_BCE, Package_TO_SOT_THT:TO-220-3_Vertical, symbol Device:Q_PNP_BCE
- added R1: 220, Resistor_THT:R_Axial_DIN0207_L6.3mm_D2.5mm_P7.62mm_Horizontal, symbol Device:R
- added R13: 100k, Resistor_THT:R_Axial_DIN0207_L6.3mm_D2.5mm_P7.62mm_Horizontal, symbol Device:R
- C1: footprint Capacitor_THT:CP_Radial_D10.0mm_P2.50mm -> Capacitor_THT:C_Disc_D5.0mm_W2.5mm_P5.00mm
- C2: footprint Capacitor_THT:CP_Radial_D10.0mm_P2.50mm -> Capacitor_THT:C_Disc_D6.0mm_W2.5mm_P5.00mm
- R12: value 150 -> 2.2k
Connections:
- net GNDREF: now also D1.2 (A), OUT-1.1, Q3.1 (E)
- net PWR: now also Q4.3 (E), R13.1; no longer R7.2
- net at R2.1, R3.1: now also Q3.2 (B)
- new net: Q4.2 (C), R7.2
- new net: Q4.1 (B), R1.1, R13.2
- new net: Q3.3 (C), R1.2
Other:
- moved on the sheet: D1, OUT+1, OUT-1, R2, R3, R7
Changed lines of the file:
@@
 L Device:R R2
 U 1 1 60065658
-P 6800 3400
-F 0 "R2" V 6593 3400 50  0000 C CNN
-F 1 "2.2k" V 6684 3400 50  0000 C CNN
-F 2 "Resistor_THT:R_Axial_DIN0207_L6.3mm_D2.5mm_P7.62mm_Horizontal" V 6730 3400 50  0001 C CNN
-F 3 "~" H 6800 3400 50  0001 C CNN
-	1    6800 3400
+P 7000 3400
+F 0 "R2" V 6793 3400 50  0000 C CNN
+F 1 "2.2k" V 6884 3400 50  0000 C CNN
+F 2 "Resistor_THT:R_Axial_DIN0207_L6.3mm_D2.5mm_P7.62mm_Horizontal" V 6930 3400 50  0001 C CNN
+F 3 "~" H 7000 3400 50  0001 C CNN
+	1    7000 3400
 	0    1    1    0
-$EndComp
-$Comp
-L Device:Q_NPN_BCE Q2
-U 1 1 6006D052
-P 7550 3400
-F 0 "Q2" H 7741 3446 50  0000 L CNN
-F 1 "TIP31C" H 7741 3355 50  0000 L CNN
-F 2 "Package_TO_SOT_THT:TO-220-3_Vertical" H 7750 3500 50  0001 C CNN
-F 3 "~" H 7550 3400 50  0001 C CNN
-	1    7550 3400
-	1    0    0    -1
 $EndComp
 $Comp
 L power:GNDREF #PWR0101
 U 1 1 6006FF68
-P 7400 3800
-F 0 "#PWR0101" H 7400 3550 50  0001 C CNN
-F 1 "GNDREF" H 7405 3627 50  0000 C CNN
-F 2 "" H 7400 3800 50  0001 C CNN
-F 3 "" H 7400 3800 50  0001 C CNN
-	1    7400 3800
+P 7700 3800
+F 0 "#PWR0101" H 7700 3550 50  0001 C CNN
+F 1 "GNDREF" H 7705 3627 50  0000 C CNN
+F 2 "" H 7700 3800 50  0001 C CNN
+F 3 "" H 7700 3800 50  0001 C CNN
+	1    7700 3800
 	1    0    0    -1
 $EndComp
@@
 Wire Wire Line
 	6050 3950 6550 3950
-Text GLabel 7600 2550 0    50   Input ~ 0
+Text GLabel 8850 2400 1    50   Input ~ 0
 PWR
 $Comp
 L Device:R R7
 U 1 1 6009AF9C
-P 7750 2550
-F 0 "R7" V 7543 2550 50  0000 C CNN
-F 1 "10" V 7634 2550 50  0000 C CNN
-F 2 "Resistor_THT:R_Axial_DIN0516_L15.5mm_D5.0mm_P20.32mm_Horizontal" V 7680 2550 50  0001 C CNN
-F 3 "~" H 7750 2550 50  0001 C CNN
-	1    7750 2550
-	0    1    1    0
+P 8850 3300
+F 0 "R7" V 8643 3300 50  0000 C CNN
+F 1 "10" V 8734 3300 50  0000 C CNN
+F 2 "Resistor_THT:R_Axial_DIN0516_L15.5mm_D5.0mm_P20.32mm_Horizontal" V 8780 3300 50  0001 C CNN
+F 3 "~" H 8850 3300 50  0001 C CNN
+	1    8850 3300
+	-1   0    0    1
 $EndComp
 $Comp
@@
 L speaker-switcher-remote-rescue:spade-terminal-arduino OUT-1
 U 1 1 600B4492
-P 8700 3000
-F 0 "OUT-1" H 8778 3035 50  0000 L CNN
-F 1 "spade-terminal" H 8800 2950 30  0000 L CNN
-F 2 "arduino-nano:SpadeTerminal635" H 8550 3150 50  0001 C CNN
-F 3 "" H 8550 3150 50  0001 C CNN
-	1    8700 3000
+P 9350 3800
+F 0 "OUT-1" H 9428 3835 50  0000 L CNN
+F 1 "spade-terminal" H 9450 3750 30  0000 L CNN
+F 2 "arduino-nano:SpadeTerminal635" H 9200 3950 50  0001 C CNN
+F 3 "" H 9200 3950 50  0001 C CNN
+	1    9350 3800
 	1    0    0    -1
 $EndComp
@@
 L speaker-switcher-remote-rescue:spade-terminal-arduino OUT+1
 U 1 1 600B4885
-P 8700 2900
-F 0 "OUT+1" H 8778 2935 50  0000 L CNN
-F 1 "spade-terminal" H 8800 3050 30  0000 L CNN
-F 2 "arduino-nano:SpadeTerminal635" H 8550 3050 50  0001 C CNN
-F 3 "" H 8550 3050 50  0001 C CNN
-	1    8700 2900
-	1    0    0    -1
-$EndComp
-Text Label 8550 2850 0    50   ~ 0
+P 9350 3700
+F 0 "OUT+1" H 9428 3735 50  0000 L CNN
+F 1 "spade-terminal" H 9450 3850 30  0000 L CNN
+F 2 "arduino-nano:SpadeTerminal635" H 9200 3850 50  0001 C CNN
+F 3 "" H 9200 3850 50  0001 C CNN
+	1    9350 3700
+	1    0    0    -1
+$EndComp
+Text Label 9200 3650 0    50   ~ 0
 OUT+
-Text Label 8550 3150 0    50   ~ 0
+Text Label 9200 3950 0    50   ~ 0
 OUT-
 $Comp
@@
 F 0 "C1" H 3668 5296 50  0000 L CNN
 F 1 ".33uF" H 3668 5205 50  0000 L CNN
-F 2 "Capacitor_THT:CP_Radial_D10.0mm_P2.50mm" H 3588 5100 50  0001 C CNN
+F 2 "Capacitor_THT:C_Disc_D5.0mm_W2.5mm_P5.00mm" H 3588 5100 50  0001 C CNN
 F 3 "~" H 3550 5250 50  0001 C CNN
 	1    3550 5250
@@
 F 0 "C2" H 4768 5296 50  0000 L CNN
 F 1 ".1uF" H 4768 5205 50  0000 L CNN
-F 2 "Capacitor_THT:CP_Radial_D10.0mm_P2.50mm" H 4688 5100 50  0001 C CNN
+F 2 "Capacitor_THT:C_Disc_D6.0mm_W2.5mm_P5.00mm" H 4688 5100 50  0001 C CNN
 F 3 "~" H 4650 5250 50  0001 C CNN
 	1    4650 5250
@@
 Wire Wire Line
 	5650 3050 6300 3050
-Wire Wire Line
-	8400 2550 8400 2900
-Wire Wire Line
-	8400 2900 8600 2900
-Wire Wire Line
-	8600 3000 8400 3000
-Wire Wire Line
-	8400 3000 8400 3200
-Wire Wire Line
-	8400 3200 8050 3200
 $Comp
 L Device:D D1
 U 1 1 60218F13
-P 8050 2850
-F 0 "D1" V 8004 2929 50  0000 L CNN
-F 1 "1N4148" H 7900 2750 50  0000 L CNN
-F 2 "Diode_THT:D_DO-41_SOD81_P7.62mm_Horizontal" H 8050 2850 50  0001 C CNN
-F 3 "~" H 8050 2850 50  0001 C CNN
-	1    8050 2850
+P 8650 3750
+F 0 "D1" V 8604 3829 50  0000 L CNN
+F 1 "1N4148" H 8500 3650 50  0000 L CNN
+F 2 "Diode_THT:D_DO-41_SOD81_P7.62mm_Horizontal" H 8650 3750 50  0001 C CNN
+F 3 "~" H 8650 3750 50  0001 C CNN
+	1    8650 3750
 	0    1    1    0
 $EndComp
-Connection ~ 8050 2550
-Wire Wire Line
-	8050 2550 8400 2550
-Wire Wire Line
-	8050 2550 8050 2700
-Wire Wire Line
-	8050 3000 8050 3200
-Connection ~ 8050 3200
-Wire Wire Line
-	8050 3200 7650 3200
-Wire Wire Line
-	7900 2550 8050 2550
-Wire Wire Line
-	7650 3600 7650 3800
-Wire Wire Line
-	7650 3800 7400 3800
 Wire Wire Line
 	6550 3400 6550 3950
@@
 Wire Wire Line
 	7050 4900 7300 4900
-Connection ~ 7400 3800
-Wire Wire Line
-	7100 3800 7400 3800
-Wire Wire Line
-	7100 3800 7100 3750
-Wire Wire Line
-	7100 3400 7100 3450
-Wire Wire Line
-	7350 3400 7100 3400
-Connection ~ 7100 3400
-Wire Wire Line
-	6950 3400 7100 3400
+Connection ~ 7700 3800
+Wire Wire Line
+	7400 3800 7700 3800
+Wire Wire Line
+	7400 3800 7400 3750
+Wire Wire Line
+	7400 3400 7400 3450
+Connection ~ 7400 3400
+Wire Wire Line
+	7150 3400 7400 3400
 $Comp
 L Device:R R3
 U 1 1 6006F615
-P 7100 3600
-F 0 "R3" H 7170 3646 50  0000 L CNN
-F 1 "10k" H 7170 3555 50  0000 L CNN
-F 2 "Resistor_THT:R_Axial_DIN0207_L6.3mm_D2.5mm_P7.62mm_Horizontal" V 7030 3600 50  0001 C CNN
-F 3 "~" H 7100 3600 50  0001 C CNN
-	1    7100 3600
-	1    0    0    -1
-$EndComp
-Wire Wire Line
-	6650 3400 6550 3400
+P 7400 3600
+F 0 "R3" H 7470 3646 50  0000 L CNN
+F 1 "10k" H 7470 3555 50  0000 L CNN
+F 2 "Resistor_THT:R_Axial_DIN0207_L6.3mm_D2.5mm_P7.62mm_Horizontal" V 7330 3600 50  0001 C CNN
+F 3 "~" H 7400 3600 50  0001 C CNN
+	1    7400 3600
+	1    0    0    -1
+$EndComp
+Wire Wire Line
+	6850 3400 6550 3400
 $Comp
 L Device:R R9
@@
 P 6800 2350
 F 0 "R12" H 6870 2396 50  0000 L CNN
-F 1 "150" H 6870 2305 50  0000 L CNN
+F 1 "2.2k" H 6870 2305 50  0000 L CNN
 F 2 "Resistor_THT:R_Axial_DIN0207_L6.3mm_D2.5mm_P7.62mm_Horizontal" V 6730 2350 50  0001 C CNN
 F 3 "~" H 6800 2350 50  0001 C CNN
@@
 	1    0    0    -1
 $EndComp
+$Comp
+L Device:Q_PNP_BCE Q4
+U 1 1 60427C3F
+P 8750 2950
+F 0 "Q4" H 8940 2950 50  0000 L CNN
+F 1 "Q_PNP_BCE" H 8940 2995 50  0001 L CNN
+F 2 "Package_TO_SOT_THT:TO-220-3_Vertical" H 8950 3050 50  0001 C CNN
+F 3 "~" H 8750 2950 50  0001 C CNN
+	1    8750 2950
+	1    0    0    1
+$EndComp
+Wire Wire Line
+	8850 3450 8850 3600
+$Comp
+L power:GNDREF #PWR0103
+U 1 1 60454D62
+P 8850 4000
+F 0 "#PWR0103" H 8850 3750 50  0001 C CNN
+F 1 "GNDREF" H 8855 3827 50  0000 C CNN
+F 2 "" H 8850 4000 50  0001 C CNN
+F 3 "" H 8850 4000 50  0001 C CNN
+	1    8850 4000
+	1    0    0    -1
+$EndComp
+Wire Wire Line
+	8850 3800 8850 3900
+Wire Wire Line
+	8850 3700 9250 3700
+Wire Wire Line
+	8850 3800 9250 3800
+$Comp
+L Device:Q_NPN_EBC Q3
+U 1 1 604698E0
+P 7850 3400
+F 0 "Q3" V 8150 3350 50  0000 L CNN
+F 1 "2N2222" V 8050 3250 50  0000 L CNN
+F 2 "Package_TO_SOT_THT:TO-92" H 8050 3500 50  0001 C CNN
+F 3 "~" H 7850 3400 50  0001 C CNN
+	1    7850 3400
+	1    0    0    -1
+$EndComp
+$Comp
+L Device:R R1
+U 1 1 6046C227
+P 8100 2950
+F 0 "R1" V 7893 2950 50  0000 C CNN
+F 1 "220" V 7984 2950 50  0000 C CNN
+F 2 "Resistor_THT:R_Axial_DIN0207_L6.3mm_D2.5mm_P7.62mm_Horizontal" V 8030 2950 50  0001 C CNN
+F 3 "~" H 8100 2950 50  0001 C CNN
+	1    8100 2950
+	0    1    1    0
+$EndComp
+Wire Wire Line
+	7950 2950 7950 3200
+Wire Wire Line
+	7950 3600 7950 3800
+Wire Wire Line
+	7700 3800 7950 3800
+Wire Wire Line
+	7400 3400 7650 3400
+Wire Wire Line
+	8650 3600 8850 3600
+Connection ~ 8850 3600
+Wire Wire Line
+	8850 3600 8850 3700
+Wire Wire Line
+	8650 3900 8850 3900
+Connection ~ 8850 3900
+Wire Wire Line
+	8850 3900 8850 4000
+Wire Wire Line
+	8250 2950 8400 2950
+$Comp
+L Device:R R13
+U 1 1 6042AFE2
+P 8400 2700
+F 0 "R13" H 8470 2746 50  0000 L CNN
+F 1 "100k" H 8470 2655 50  0000 L CNN
+F 2 "Resistor_THT:R_Axial_DIN0207_L6.3mm_D2.5mm_P7.62mm_Horizontal" V 8330 2700 50  0001 C CNN
+F 3 "~" H 8400 2700 50  0001 C CNN
+	1    8400 2700
+	1    0    0    -1
+$EndComp
+Wire Wire Line
+	8850 2500 8850 2750
+Wire Wire Line
+	8400 2500 8850 2500
+Wire Wire Line
+	8850 2400 8850 2500
+Connection ~ 8850 2500
+Wire Wire Line
+	8400 2550 8400 2500
+Wire Wire Line
+	8400 2850 8400 2950
+Connection ~ 8400 2950
+Wire Wire Line
+	8400 2950 8550 2950
 $EndSCHEMATC
